File: PowerBoard.kicad_sch (KiCad schematic)
At the start: 15 parts, among them J26 Power to TopBoard, J27 Power to TopBoard, J28 Power to TopBoard, J29 Power from BackBoard, U21 LT1085CM-3.3#PBF

Commit message: Lidar基板Rev.2発注
Other:
- company: (none) -> Fornax
- title: (none) -> PowerBoard Rev.1
Changed lines of the file:
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@@
 	(generator_version "8.0")
 	(paper "A5")
+	(title_block
+		(title "PowerBoard Rev.1")
+		(rev "1")
+		(company "Fornax")
+	)
 	(junction
 		(at 118.11 74.93)

Commit message: メイン基板Rev.2完成
Parts:
- renumbered C75 to C65, C76 to C66, C77 to C67, C78 to C68, J26 to J30, J27 to J31, J28 to J32, J29 to J33, MD2 to MD1, R43 to R45, R44 to R46, R45 to R47, R46 to R48, R47 to R49, U21 to U24
