File: TopBoard.kicad_sch (KiCad schematic)
At the start: 83 parts, among them J1 Power from PowerBoard, J10 UnitV02, J11 GH-S37D, J12 NeoPixel, J13 LoadCell, J14 NeoPixel, J15 LoadCell, J2 Power from PowerBoard, J3 ST-Link, J4 Power from PowerBoard, J5 Com from BackBoard, J6 to TileBoard, J7 to LidarBoard, J8 UnitV01, J9 GH-S37D, Q1 BSS138, Q2 BSS138, Q3 BSS138, Q4 BSS138, SW1 RESET_SWITCH, SW2 MODE_SWITCH, U1 VL53L0X, U2 Sit2001B, U3 VL53L0X, U4 STM32H747IGT6, U5 AE-BNO055-BO, U6 NJU77551F, U7 NJU77551F

Commit message: after ordered TileBoard Rev.1 and PowerBoard Rev.1
Parts:
- C1, C10, C11, C12, C13, C14, C15, C16, C17, C18, C19, C2, C20, C21, C22, C23, C24, C25, C26, C27, C28, C29, C3, C30, C31, C4, C5, C6, C7, C8, C9: footprint Capacitor_SMD:C_0402_1005Metric -> Capacitor_SMD:C_0603_1608Metric
- R1, R10, R11, R12, R13, R14, R15, R16, R17, R18, R19, R2, R20, R3, R4, R5, R6, R7, R8, R9: footprint Capacitor_SMD:C_0402_1005Metric -> Resistor_SMD:R_0603_1608Metric
Connections:
- net SWO: no longer J3.8 (JTDO/SWO)
- no-connect marks 93 -> 94
Changed lines of the file:
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@@
 	)
 	(no_connect
+		(at 146.05 35.56)
+	)
+	(no_connect
 		(at 267.97 142.24)
 	)
@@
 	(wire
 		(pts
-			(xy 146.05 35.56) (xy 147.32 35.56)
-		)
-		(stroke
-			(width 0)
-			(type default)
-		)
-	)
-	(wire
-		(pts
 			(xy 228.6 25.4) (xy 238.76 25.4)
 		)
@@
 		)
 	)
-	(label "SWO"
-		(at 147.32 35.56 0)
-		(fields_autoplaced yes)
-		(effects
-			(font
-				(size 1.27 1.27)
-			)
-			(justify left bottom)
-		)
-	)
 	(label "SDA"
 		(at 31.75 184.15 180)
@@
 			)
 		)
-		(property "Footprint" "Capacitor_SMD:C_0402_1005Metric"
+		(property "Footprint" "Resistor_SMD:R_0603_1608Metric"
 			(at 248.92 70.358 90)
 			(effects
@@
 			)
 		)
-		(property "Footprint" "Capacitor_SMD:C_0402_1005Metric"
+		(property "Footprint" "Capacitor_SMD:C_0603_1608Metric"
 			(at 260.0452 25.4 0)
 			(effects
@@
 			)
 		)
-		(property "Footprint" "Capacitor_SMD:C_0402_1005Metric"
+		(property "Footprint" "Resistor_SMD:R_0603_1608Metric"
 			(at 121.412 224.79 90)
 			(effects
@@
 			)
 		)
-		(property "Footprint" "Capacitor_SMD:C_0402_1005Metric"
+		(property "Footprint" "Capacitor_SMD:C_0603_1608Metric"
 			(at 220.6752 137.16 0)
 			(effects
@@
 			)
 		)
-		(property "Footprint" "Capacitor_SMD:C_0402_1005Metric"
+		(property "Footprint" "Capacitor_SMD:C_0603_1608Metric"
 			(at 216.8652 92.71 0)
 			(effects
@@
 			)
 		)
-		(property "Footprint" "Capacitor_SMD:C_0402_1005Metric"
+		(property "Footprint" "Resistor_SMD:R_0603_1608Metric"
 			(at 261.62 62.738 90)
 			(effects
@@
 			)
 		)
-		(property "Footprint" "Capacitor_SMD:C_0402_1005Metric"
+		(property "Footprint" "Resistor_SMD:R_0603_1608Metric"
 			(at 48.26 271.018 90)
 			(effects
@@
 			)
 		)
-		(property "Footprint" "Capacitor_SMD:C_0402_1005Metric"
+		(property "Footprint" "Capacitor_SMD:C_0603_1608Metric"
 			(at 371.8052 25.4 0)
 			(effects
@@
 			)
 		)
-		(property "Footprint" "Capacitor_SMD:C_0402_1005Metric"
+		(property "Footprint" "Capacitor_SMD:C_0603_1608Metric"
 			(at 341.3252 25.4 0)
 			(effects
@@
 			)
 		)
-		(property "Footprint" "Capacitor_SMD:C_0402_1005Metric"
+		(property "Footprint" "Capacitor_SMD:C_0603_1608Metric"
 			(at 209.2452 25.4 0)
 			(effects
@@
 			)
 		)
-		(property "Footprint" "Capacitor_SMD:C_0402_1005Metric"
+		(property "Footprint" "Capacitor_SMD:C_0603_1608Metric"
 			(at 350.2152 50.8 0)
 			(effects
@@
 			)
 		)
-		(property "Footprint" "Capacitor_SMD:C_0402_1005Metric"
+		(property "Footprint" "Capacitor_SMD:C_0603_1608Metric"
 			(at 188.9252 25.4 0)
 			(effects
@@
 			)
 		)
-		(property "Footprint" "Capacitor_SMD:C_0402_1005Metric"
+		(property "Footprint" "Capacitor_SMD:C_0603_1608Metric"
 			(at 280.3652 25.4 0)
 			(effects
@@
 			)
 		)
-		(property "Footprint" "Capacitor_SMD:C_0402_1005Metric"
+		(property "Footprint" "Resistor_SMD:R_0603_1608Metric"
 			(at 136.652 250.19 90)
 			(effects
@@
 			)
 		)
-		(property "Footprint" "Capacitor_SMD:C_0402_1005Metric"
+		(property "Footprint" "Resistor_SMD:R_0603_1608Metric"
 			(at 48.26 237.998 90)
 			(effects
@@
 			)
 		)
-		(property "Footprint" "Capacitor_SMD:C_0402_1005Metric"
+		(property "Footprint" "Capacitor_SMD:C_0603_1608Metric"
 			(at 224.4852 92.71 0)
 			(effects
@@
 			)
 		)
-		(property "Footprint" "Capacitor_SMD:C_0402_1005Metric"
+		(property "Footprint" "Capacitor_SMD:C_0603_1608Metric"
 			(at 321.0052 25.4 0)
 			(effects
@@
 			)
 		)
-		(property "Footprint" "Capacitor_SMD:C_0402_1005Metric"
+		(property "Footprint" "Resistor_SMD:R_0603_1608Metric"
 			(at 48.26 268.478 90)
 			(effects
@@
 			)
 		)
-		(property "Footprint" "Capacitor_SMD:C_0402_1005Metric"
+		(property "Footprint" "Resistor_SMD:R_0603_1608Metric"
 			(at 112.522 87.63 90)
 			(effects
@@
 			)
 		)
-		(property "Footprint" "Capacitor_SMD:C_0402_1005Metric"
+		(property "Footprint" "Resistor_SMD:R_0603_1608Metric"
 			(at 80.772 233.68 90)
 			(effects
@@
 			)
 		)
-		(property "Footprint" "Capacitor_SMD:C_0402_1005Metric"
+		(property "Footprint" "Capacitor_SMD:C_0603_1608Metric"
 			(at 342.5952 50.8 0)
 			(effects
@@
 			)
 		)
-		(property "Footprint" "Capacitor_SMD:C_0402_1005Metric"
+		(property "Footprint" "Resistor_SMD:R_0603_1608Metric"
 			(at 75.692 184.15 90)
 			(effects
@@
 			)
 		)
-		(property "Footprint" "Capacitor_SMD:C_0402_1005Metric"
+		(property "Footprint" "Capacitor_SMD:C_0603_1608Metric"
 			(at 392.1252 25.4 0)
 			(effects
@@
 			)
 		)
-		(property "Footprint" "Capacitor_SMD:C_0402_1005Metric"
+		(property "Footprint" "Capacitor_SMD:C_0603_1608Metric"
 			(at 265.43 51.1048 0)
 			(effects
@@
 			)
 		)
-		(property "Footprint" "Capacitor_SMD:C_0402_1005Metric"
+		(property "Footprint" "Capacitor_SMD:C_0603_1608Metric"
 			(at 256.54 246.6848 0)
 			(effects
@@
 			)
 		)
-		(property "Footprint" "Capacitor_SMD:C_0402_1005Metric"
+		(property "Footprint" "Capacitor_SMD:C_0603_1608Metric"
 			(at 256.54 237.7948 0)
 			(effects
@@
 			)
 		)
-		(property "Footprint" "Capacitor_SMD:C_0402_1005Metric"
+		(property "Footprint" "Capacitor_SMD:C_0603_1608Metric"
 			(at 210.5152 137.16 0)
 			(effects
@@
 			)
 		)
-		(property "Footprint" "Capacitor_SMD:C_0402_1005Metric"
+		(property "Footprint" "Capacitor_SMD:C_0603_1608Metric"
 			(at 229.5652 25.4 0)
 			(effects
@@
 			)
 		)
-		(property "Footprint" "Capacitor_SMD:C_0402_1005Metric"
+		(property "Footprint" "Resistor_SMD:R_0603_1608Metric"
 			(at 97.282 87.63 90)
 			(effects
@@
 			)
 		)
-		(property "Footprint" "Capacitor_SMD:C_0402_1005Metric"
+		(property "Footprint" "Capacitor_SMD:C_0603_1608Metric"
 			(at 219.4052 25.4 0)
 			(effects
@@
 			)
 		)
-		(property "Footprint" "Capacitor_SMD:C_0402_1005Metric"
+		(property "Footprint" "Resistor_SMD:R_0603_1608Metric"
 			(at 136.652 224.79 90)
 			(effects
@@
 			)
 		)
-		(property "Footprint" "Capacitor_SMD:C_0402_1005Metric"
+		(property "Footprint" "Capacitor_SMD:C_0603_1608Metric"
 			(at 290.5252 25.4 0)
 			(effects
@@
 			)
 		)
-		(property "Footprint" "Capacitor_SMD:C_0402_1005Metric"
+		(property "Footprint" "Resistor_SMD:R_0603_1608Metric"
 			(at 56.642 273.05 90)
 			(effects
@@
 			)
 		)
-		(property "Footprint" "Capacitor_SMD:C_0402_1005Metric"
+		(property "Footprint" "Resistor_SMD:R_0603_1608Metric"
 			(at 229.87 83.058 90)
 			(effects
@@
 			)
 		)
-		(property "Footprint" "Capacitor_SMD:C_0402_1005Metric"
+		(property "Footprint" "Capacitor_SMD:C_0603_1608Metric"
 			(at 381.9652 25.4 0)
 			(effects
@@
 			)
 		)
-		(property "Footprint" "Capacitor_SMD:C_0402_1005Metric"
+		(property "Footprint" "Capacitor_SMD:C_0603_1608Metric"
 			(at 199.0852 25.4 0)
 			(effects
@@
 			)
 		)
-		(property "Footprint" "Capacitor_SMD:C_0402_1005Metric"
+		(property "Footprint" "Capacitor_SMD:C_0603_1608Metric"
 			(at 310.8452 25.4 0)
 			(effects
@@
 			)
 		)
-		(property "Footprint" "Capacitor_SMD:C_0402_1005Metric"
+		(property "Footprint" "Resistor_SMD:R_0603_1608Metric"
 			(at 121.412 250.19 90)
 			(effects
@@
 			)
 		)
-		(property "Footprint" "Capacitor_SMD:C_0402_1005Metric"
+		(property "Footprint" "Capacitor_SMD:C_0603_1608Metric"
 			(at 300.6852 25.4 0)
 			(effects
@@
 			)
 		)
-		(property "Footprint" "Capacitor_SMD:C_0402_1005Metric"
+		(property "Footprint" "Capacitor_SMD:C_0603_1608Metric"
 			(at 331.1652 25.4 0)
 			(effects
@@
 			)
 		)
-		(property "Footprint" "Capacitor_SMD:C_0402_1005Metric"
+		(property "Footprint" "Capacitor_SMD:C_0603_1608Metric"
 			(at 402.2852 25.4 0)
 			(effects
@@
 			)
 		)
-		(property "Footprint" "Capacitor_SMD:C_0402_1005Metric"
+		(property "Footprint" "Resistor_SMD:R_0603_1608Metric"
 			(at 248.92 75.438 90)
 			(effects
@@
 			)
 		)
-		(property "Footprint" "Capacitor_SMD:C_0402_1005Metric"
+		(property "Footprint" "Resistor_SMD:R_0603_1608Metric"
 			(at 90.932 184.15 90)
 			(effects
@@
 			)
 		)
-		(property "Footprint" "Capacitor_SMD:C_0402_1005Metric"
+		(property "Footprint" "Capacitor_SMD:C_0603_1608Metric"
 			(at 249.8852 25.4 0)
 			(effects
@@
 			)
 		)
-		(property "Footprint" "Capacitor_SMD:C_0402_1005Metric"
+		(property "Footprint" "Capacitor_SMD:C_0603_1608Metric"
 			(at 351.4852 25.4 0)
 			(effects
@@
 			)
 		)
-		(property "Footprint" "Capacitor_SMD:C_0402_1005Metric"
+		(property "Footprint" "Resistor_SMD:R_0603_1608Metric"
 			(at 56.642 242.57 90)
 			(effects
@@
 			)
 		)
-		(property "Footprint" "Capacitor_SMD:C_0402_1005Metric"
+		(property "Footprint" "Capacitor_SMD:C_0603_1608Metric"
 			(at 361.6452 25.4 0)
 			(effects
@@
 			)
 		)
-		(property "Footprint" "Capacitor_SMD:C_0402_1005Metric"
+		(property "Footprint" "Resistor_SMD:R_0603_1608Metric"
 			(at 80.772 264.16 90)
 			(effects
@@
 			)
 		)
-		(property "Footprint" "Capacitor_SMD:C_0402_1005Metric"
+		(property "Footprint" "Capacitor_SMD:C_0603_1608Metric"
 			(at 239.7252 25.4 0)
 			(effects
@@
 			)
 		)
-		(property "Footprint" "Capacitor_SMD:C_0402_1005Metric"
+		(property "Footprint" "Resistor_SMD:R_0603_1608Metric"
 			(at 48.26 240.538 90)
 			(effects
@@
 			)
 		)
-		(property "Footprint" "Capacitor_SMD:C_0402_1005Metric"
+		(property "Footprint" "Capacitor_SMD:C_0603_1608Metric"
 			(at 270.2052 25.4 0)
 			(effects

Commit message: Lidar基板Rev.2発注
Parts:
- R11, R14, R17, R20: value 1M -> 47k
Other:
- company: (none) -> Fornax
- title: (none) -> TopBoard Rev.1
Changed lines of the file:
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@@
 	(generator_version "8.0")
 	(paper "A3")
+	(title_block
+		(title "TopBoard Rev.1")
+		(rev "1")
+		(company "Fornax")
+	)
 	(junction
 		(at 92.71 180.34)
@@
 			)
 		)
-		(property "Value" "1M"
+		(property "Value" "47k"
 			(at 81.534 233.426 0)
 			(effects
@@
 			)
 		)
-		(property "Value" "1M"
+		(property "Value" "47k"
 			(at 57.15 272.796 0)
 			(effects
@@
 			)
 		)
-		(property "Value" "1M"
+		(property "Value" "47k"
 			(at 57.15 242.316 0)
 			(effects
@@
 			)
 		)
-		(property "Value" "1M"
+		(property "Value" "47k"
 			(at 81.534 263.906 0)
 			(effects

Commit message: メイン基板Rev.2完成
Parts:
- removed C18, C19, C22, C24, C25, C27: 0.1uF, Capacitor_SMD:C_0603_1608Metric, symbol Device:C
- removed C23, C26: 1uF, Capacitor_SMD:C_0603_1608Metric, symbol Device:C
- removed C30, C31: 2.2uF, Capacitor_SMD:C_0603_1608Metric, symbol Device:C
- removed J12, J14: NeoPixel, Connector_JST:JST_ZH_B3B-ZR_1x03_P1.50mm_Vertical, symbol Connector:Conn_01x03_Socket
- removed Q3, Q4: BSS138, Package_TO_SOT_SMD:SOT-23, symbol Simulation_SPICE:NMOS
- removed R10, R15, R16, R9: 10k, Resistor_SMD:R_0603_1608Metric, symbol Device:R
- removed U1, U3: VL53L0X, Connector_PinHeader_2.54mm:PinHeader_1x05_P2.54mm_Vertical, symbol VL53l0X:VL53L0X_SwScience
- removed U4: STM32H747IGT6, Package_QFP:LQFP-176_24x24mm_P0.5mm, symbol MCU_ST_STM32H7:STM32H747IGTx
- added U1, U3: ~, Connector_PinSocket_2.54mm:PinSocket_1x06_P2.54mm_Vertical, symbol VL53l0X:VL53L0X_SwScience_6pin
- added U4: STM32H723ZGTx, Package_QFP:LQFP-144_20x20mm_P0.5mm, symbol MCU_ST_STM32H7:STM32H723ZGTx
- added U7: MOUDLE-SEEEDUINO-XIAO-ESP32C3, XIAO:MOUDLE14P-SMD-2.54-21X17.8MM, symbol XIAO:MOUDLE-SEEEDUINO-XIAO-ESP32C3
- C1, C15: value 0.1uF -> 1uF
- C14: value 0.1uF -> 4.7uF
- C20, C21: value 0.1uF -> 2.2uF
- FB1: footprint Capacitor_SMD:C_0603_1608Metric -> Inductor_SMD:L_0603_1608Metric
- J11, J9: footprint Connector_PinHeader_2.54mm:PinHeader_1x03_P2.54mm_Vertical -> Connector_JST:JST_ZH_B3B-ZR_1x03_P1.50mm_Vertical
- R1, R2: footprint Resistor_SMD:R_0603_1608Metric -> Capacitor_SMD:C_0603_1608Metric_Pad1.08x0.95mm_HandSolder
- R3: value 10k -> 47
- R4: value 0 -> 10k; footprint Resistor_SMD:R_0603_1608Metric -> Capacitor_SMD:C_0603_1608Metric_Pad1.08x0.95mm_HandSolder
- renumbered C28 to C18, C29 to C19, J13 to J12, J15 to J13, R12 to R10, R13 to R11, R14 to R12, R17 to R13, R18 to R14, R19 to R15, R20 to R16, R11 to R9, U7 to U8
Connections:
- net +3.3V: now also R4.1, U1.3 (VDD), U3.3 (VDD), U4.108 (VDD), U4.121 (VDD), U4.131 (VDD), U4.144 (VDD), U4.17 (VDD), U4.30 (VDD), U4.39 (VDD), U4.52 (VDD), U4.6 (VBAT), U4.62 (VDD), U4.72 (VDD), U4.84 (VDD), U4.95 (VDD33USB); no longer C15.1, C16.1, C17.1, C20.1, C21.1, R2.1
- net +5V: now also U7.14 (5V)
- net AD1: now also U4.44 (PC4)
- net AD2: now also U4.49 (PF11)
- net AD3: now also U4.53 (PF13)
- net DIN1: now also R8.2, U4.42 (PA6); no longer R7.2
- net DIN4: now also U4.4 (PE5)
- net GND: now also C17.1, C20.1, C21.1, R2.1, U1.4 (GND), U3.4 (GND), U4.107 (VSS), U4.120 (VSS), U4.130 (VSS), U4.16 (VSS), U4.31 (VSSA), U4.38 (VSS), U4.51 (VSS), U4.61 (VSS), U4.83 (VSS), U4.94 (VSS), U7.13 (GND); no longer C17.2, C20.2, C21.2, R3.1
- net HSE: now also U4.23 (PH0)
- net NRST: now also C17.2, U4.25 (NRST)
- net PWM1: now also U4.60 (PE9)
- net PWM2: now also U4.41 (PA5)
- net RX1: now also U4.76 (PB15)
- net RX2: now also U4.37 (PA3)
- net RX3: now also U4.69 (PB10)
- net RX4: now also U4.35 (PA1)
- net RX5: now also U4.73 (PB12)
- net RX6: now also U4.97 (PC7)
- net SCL: now also U1.6 (SCL), U3.6 (SCL), U4.54 (PF14)
- net SDA: now also U1.5 (SDA), U3.5 (SDA), U4.55 (PF15)
- net SWCLK: now also U4.109 (PA14(JTCK)
- net SWDIO: now also U4.105 (PA13(JTMS)
- net TX1: now also U4.75 (PB14)
- net TX2: now also U4.36 (PA2)
- net TX3: now also U4.70 (PB11)
- net TX4: now also U4.34 (PA0)
- net TX5: now also U4.74 (PB13)
- net TX6: now also U4.96 (PC6)
- net VDDA: now also C15.1, C16.1, R3.1, U4.33 (VDDA); no longer R4.1
- net XSHUT1: now also U1.2 (XSHUT), U4.56 (PG0)
- net XSHUT2: now also U3.2 (XSHUT), U4.57 (PG1)
- net at SW2.1 (A): now also R1.2; no longer R2.2
- net at SW2.2 (B): now also U4.138 (BOOT0)
- net at R4.2: now also U4.143 (PDR_ON)
- net at D1.4 (DIN), Q2.1 (D): now also R7.2; no longer R8.2
- net at SW2.3 (C): now also R2.2; no longer R3.2
- new net: C20.2, U4.71 (VCAP)
- new net: R3.2, U4.32 (VREF+)
- new net: C21.2, U4.106 (VCAP)
- new net RX7: U4.18 (PF6), U7.7 (PB08_A6_D6_TX)
- new net TX7: U4.19 (PF7), U7.8 (PB09_A7_D7_RX)
- no-connect marks 94 -> 106
Other:
- note added: "VBAT"
- note added: "VDD"
- note added: "XIAO-ESP32"
- note added: "ZH,Vertical"
- note removed: "PinHeader,Vertical"
- title: TopBoard Rev.1 -> TopBoard Rev.2
- moved on the sheet: C18, C19, R7, U2
