File: BackBoard.kicad_sch (KiCad schematic)
At the start: 78 parts, among them J16 Power to TopBoard, J17 Comm to TopBoard, J18 Conn_01x08_Socket, J19 ST-Link, J20 USB_C_Receptacle_USB2.0_16P, M1 STS3032, M2 STS3032, M3 STS3032, M4 STS3032, Q5 TJ15S06M3L, Q6 BSS138, Q7 BSS138, SW3 GW-12LWP, SW4 RESET_SWITCH, SW5 MODE_SWITCH, SW6 START_SWITCH, SW7 RESET_SWITCH, SW8 BOOT_STRAP_SWITCH, U10 VL53L0X, U11 VL53L0X, U12 STM32F446RET6, U13 Sit2001B, U14 RP2040, U15 MAX3485, U16 W25Q128JVS, U8 MIC5219-5.0YM5-TR, U9 AZ1117CH-3.3TRG1

Commit message: Lidar基板Rev.2発注
Parts:
- removed C58: 1uF, Capacitor_SMD:C_0402_1005Metric, symbol Device:C
- removed C60: 0.1uF, Capacitor_SMD:C_0603_1608Metric_Pad1.08x0.95mm_HandSolder, symbol Device:C
- removed J20: USB_C_Receptacle_USB2.0_16P, Connector_USB:USB_C_Receptacle_G-Switch_GT-USB-7010ASV, symbol Connector:USB_C_Receptacle_USB2.0_16P
- removed SW8: BOOT_STRAP_SWITCH, SKRPACE010:SW_SKRPACE010, symbol Switch:SW_Push
- removed U14: RP2040, Package_DFN_QFN:QFN-56-1EP_7x7mm_P0.4mm_EP3.2x3.2mm, symbol MCU_RaspberryPi:RP2040
- removed U16: W25Q128JVS, Package_SO:SOIC-8_5.23x5.23mm_P1.27mm, symbol Memory_Flash:W25Q128JVS
- added J21: ST-Link, STDC14:CONN14_3220-14_CNC, symbol Connector:Conn_ST_STDC14
- added SW8: MODE_SWITCH, SSSS213202:SSSS213202, symbol Switch:SW_DPDT_x2
- added U14: STM32F446RET6, Package_QFP:LQFP-64_10x10mm_P0.5mm, symbol MCU_ST_STM32F4:STM32F446RETx
- added U16: Sit2001B, Package_TO_SOT_SMD:SOT-23-5, symbol SiT2001B:Sit2001B
- C47, C56: value 0.1uF -> 4.7uF
- C52: value 1uF -> 0.1uF
- C57: value 0.1uF -> 15pF
- R28, R29: value 20 -> 10k; footprint Capacitor_SMD:C_0402_1005Metric -> Capacitor_SMD:C_0603_1608Metric_Pad1.08x0.95mm_HandSolder
- R34: value 1k -> 680; footprint Capacitor_SMD:C_0603_1608Metric_Pad1.08x0.95mm_HandSolder -> (none)
Connections:
- net SS is gone; now on an unnamed net: R34.2
- net +3.3V: now also C47.1, C48.1, R28.1, J21.3 (VCC), U14.1 (VBAT), U14.13 (VDDA), U14.19 (VDD), U14.32 (VDD), U14.48 (VDD), U14.64 (VDD), U16.4 (VDD); no longer C54.1, C56.1, C57.1, LS1.1
- net +5V: now also LS1.1, R34.1
- net GND: now also C54.1, R29.1, J21.11 (GNDDetect), J21.5 (GND), J21.7 (GND), U14.12 (VSSA), U14.18 (VSS), U14.31 (VSS), U14.47 (VSS), U14.63 (VSS), U16.1 (GND); no longer C54.2
- net RX: now also U14.17 (PA3)
- net TX: now also U14.16 (PA2)
- net NRST2: now reaches SW7.2
- net NRST2: now also C54.2, J21.12 (~{RST}), U14.7 (NRST)
- net at R28.2: now also SW8.1 (A)
- net at R29.2: now also SW8.3 (C)
- new net: C56.1, U14.30 (VCAP_1)
- new net: SW8.2 (B), U14.60 (BOOT0)
- new net HSE2: C57.1, U14.5 (PH0), U16.5 (OUT)
- new net RX4: J21.13 (VCP_RX), U14.43 (PA10)
- new net SWCLK2: J21.6 (JCLK/SWCLK), U14.49 (PA14)
- new net SWDIO2: J21.4 (JTMS/SWDIO), U14.46 (PA13)
- new net TX4: J21.14 (VCP_TX), U14.42 (PA9)
- no-connect marks 72 -> 81
Other:
- note removed: "RP2040"
- note removed: "VREG_IN"
- company: (none) -> Fornax
- title: (none) -> BackBoard Rev.2

Commit message: LiDAR基板Rev.2修正
Parts:
- added R48: 10k, Resistor_SMD:R_0603_1608Metric, symbol Device:R
- added U23: AE-BNO055-BO, AE-BNO055-BO:AE-BNO055-BO, symbol AE-BNO055-BO:AE-BNO055-BO
- R34: footprint (none) -> Resistor_SMD:R_0603_1608Metric
Connections:
- net +3.3V: now also U23.1 (VCC)
- net CS: now also U14.41 (PA8)
- net GND: now also U23.2 (GND), U23.7 (GND)
- net MISO: now also U14.23 (PA7)
- net MOSI: now also U14.22 (PA6)
- net SCK: now also U14.21 (PA5)
- net SCL: now also U23.4 (SCL/R)
- net SDA: now also U23.3 (SDA/T)
- net at Q5.2 (G), SW3.1 (A): now also R48.1
- net at F1.2, Q5.3 (S): now also R48.2
Other:
- moved on the sheet: C47, C48, C49, C50, C51, C52, C53, C54, C55, C56, C57, J21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

Commit message: メイン基板Rev.2完成
Parts:
- removed Q7: BSS138, Package_TO_SOT_SMD:SOT-23, symbol Simulation_SPICE:NMOS
- removed R23: 10k, Capacitor_SMD:C_0603_1608Metric_Pad1.08x0.95mm_HandSolder, symbol Device:R
- removed SW3: GW-12LWP, GW-12LWP:GW-12LWP, symbol Switch:SW_DPDT_x2
- removed SW6: START_SWITCH, 100SP1T1B4M2QE:SW_100SP1T1B4M2QE, symbol Switch:SW_DPDT_x2
- removed U10, U11: VL53L0X, Connector_PinHeader_2.54mm:PinHeader_1x05_P2.54mm_Vertical, symbol VL53l0X:VL53L0X_SwScience
- added D4: LED, LED_SMD:LED_0603_1608Metric, symbol Device:LED
- added Q5: BSS138, Package_TO_SOT_SMD:SOT-23, symbol Simulation_SPICE:NMOS
- added R18: 470, Resistor_SMD:R_0603_1608Metric, symbol Device:R
- added R19: 1k, Resistor_SMD:R_0603_1608Metric, symbol Device:R
- added R25: 10k, Capacitor_SMD:C_0603_1608Metric_Pad1.08x0.95mm_HandSolder, symbol Device:R
- added SW3, SW6: B-12CCP, B-12CCP:B-12CCP, symbol B-12CCP:B-12CCP
- added U11, U13: ~, Connector_PinSocket_2.54mm:PinSocket_1x06_P2.54mm_Vertical, symbol VL53l0X:VL53L0X_SwScience_6pin
- R26: value 10k -> 1k; footprint Capacitor_SMD:C_0603_1608Metric_Pad1.08x0.95mm_HandSolder -> Resistor_SMD:R_0603_1608Metric
- renumbered C32 to C22, C33 to C23, C34 to C24, C35 to C25, C36 to C26, C37 to C27, C38 to C28, C39 to C29, C40 to C30, C41 to C31, C42 to C32, C43 to C33, C44 to C34, C45 to C35, C46 to C36, C47 to C37, C48 to C38, C49 to C39, C50 to C40, C51 to C41, C52 to C42, C53 to C43, C54 to C44, C55 to C45, C59 to C46, C57 to C47, C56 to C48, D4 to D5, D5 to D6, D6 to D7, J16 to J14, J17 to J15, J18 to J16, J19 to J17, J21 to J18, Q5 to Q3, Q6 to Q4, R48 to R17, R21 to R20, R22 to R21, R34 to R22, R25 to R23, R35 to R34, U9 to U10, U23 to U12, U12 to U14, U13 to U15, U14 to U16, U16 to U17, U15 to U18, U8 to U9
Connections:
- net +3.3V: now also Q5.2 (G), R25.1, U11.3 (VDD), U13.3 (VDD); no longer R24.1
- net +5V: now also R24.1
- net +7.5V: now also R26.2, R18.1, R19.2
- net DC: now also U16.26 (PB0)
- net DIN: now also U16.28 (PB2), Q5.3 (S), R25.2
- net GND: now also D4.1 (K), SW3.2 (B), SW3.6 (K), SW6.3 (C), SW6.6 (K), U11.4 (GND), U13.4 (GND); no longer R26.1
- net PWM: now also U16.27 (PB1)
- net SCL: now also U11.6 (SCL), U13.6 (SCL)
- net SDA: now also U11.5 (SDA), U13.5 (SDA)
- net XSHUT1: now also U13.2 (XSHUT)
- net XSHUT2: now also U11.2 (XSHUT)
- net at Q3.2 (G), R17.1: now also SW3.1 (A)
- net at D5.4 (DIN), R24.2: now also Q5.1 (D)
- net at U14.33 (PB12): now also SW6.2 (B)
- net at R23.2: now also SW6.1 (A)
- new net: D4.2 (A), R18.2
- new net: R19.1, SW3.5 (A)
- new net: R26.1, SW6.5 (A)
- no-connect marks 81 -> 86
Other:
- moved on the sheet: J14, J15, R23

Commit message: 後ろ基板Rev.2完成
Parts:
- R18: value 470 -> 680
- R26: value 1k -> 470
Connections:
- net +7.5V: no longer R26.2
- net at U14.34 (PB13): now also R26.2
- net SWO: no longer names the net of U14.55 (PB3)
- net SWO: no longer J17.8 (JTDO/SWO)
- no-connect marks 86 -> 87
Other:
- note added: "STM32 for UI"
Changed lines of the file:
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@@
 	)
 	(no_connect
+		(at 278.13 115.57)
+	)
+	(no_connect
 		(at 127 251.46)
 	)
@@
 	)
 	(no_connect
-		(at 278.13 138.43)
+		(at 149.86 132.08)
 	)
 	(no_connect
@@
 	(wire
 		(pts
-			(xy 300.99 142.24) (xy 302.26 142.24)
-		)
-		(stroke
-			(width 0)
-			(type default)
-		)
-	)
-	(wire
-		(pts
 			(xy 278.13 87.63) (xy 279.4 87.63)
 		)
@@
 	(wire
 		(pts
-			(xy 149.86 132.08) (xy 151.13 132.08)
-		)
-		(stroke
-			(width 0)
-			(type default)
-		)
-	)
-	(wire
-		(pts
 			(xy 88.9 256.54) (xy 91.44 256.54)
 		)
@@
 	(wire
 		(pts
+			(xy 300.99 142.24) (xy 300.99 148.59)
+		)
+		(stroke
+			(width 0)
+			(type default)
+		)
+	)
+	(wire
+		(pts
+			(xy 279.4 138.43) (xy 278.13 138.43)
+		)
+		(stroke
+			(width 0)
+			(type default)
+		)
+	)
+	(wire
+		(pts
 			(xy 302.26 129.54) (xy 306.07 129.54)
 		)
@@
 	(wire
 		(pts
+			(xy 300.99 148.59) (xy 279.4 148.59)
+		)
+		(stroke
+			(width 0)
+			(type default)
+		)
+	)
+	(wire
+		(pts
 			(xy 41.91 135.89) (xy 46.99 135.89)
 		)
@@
 	(wire
 		(pts
-			(xy 278.13 115.57) (xy 279.4 115.57)
-		)
-		(stroke
-			(width 0)
-			(type default)
-		)
-	)
-	(wire
-		(pts
 			(xy 240.03 130.81) (xy 242.57 130.81)
 		)
@@
 	(wire
 		(pts
+			(xy 279.4 148.59) (xy 279.4 138.43)
+		)
+		(stroke
+			(width 0)
+			(type default)
+		)
+	)
+	(wire
+		(pts
 			(xy 250.19 36.83) (xy 261.62 36.83)
 		)
@@
 		)
 	)
+	(text "STM32 for UI"
+		(exclude_from_sim no)
+		(at 25.4 162.814 0)
+		(effects
+			(font
+				(size 2.54 2.54)
+			)
+		)
+	)
 	(text "VDDA"
 		(exclude_from_sim no)
@@
 		)
 	)
-	(label "SWO"
-		(at 151.13 132.08 0)
-		(fields_autoplaced yes)
-		(effects
-			(font
-				(size 1.27 1.27)
-			)
-			(justify left bottom)
-		)
-	)
 	(label "SCL"
 		(at 279.4 85.09 0)
@@
 		)
 	)
-	(label "SWO"
-		(at 279.4 115.57 0)
-		(fields_autoplaced yes)
-		(effects
-			(font
-				(size 1.27 1.27)
-			)
-			(justify left bottom)
-		)
-	)
 	(label "RX"
 		(at 128.27 198.12 0)
@@
 	)
 	(symbol
-		(lib_id "power:+7.5V")
-		(at 302.26 142.24 0)
-		(unit 1)
-		(exclude_from_sim no)
-		(in_bom yes)
-		(on_board yes)
-		(dnp no)
-		(property "Reference" "#PWR0105"
-			(at 302.26 146.05 0)
-			(effects
-				(font
-					(size 1.27 1.27)
-				)
-				(hide yes)
-			)
-		)
-		(property "Value" "+7.5V"
-			(at 305.308 140.97 0)
-			(effects
-				(font
-					(size 1.27 1.27)
-				)
-			)
-		)
-		(property "Footprint" ""
-			(at 302.26 142.24 0)
-			(effects
-				(font
-					(size 1.27 1.27)
-				)
-				(hide yes)
-			)
-		)
-		(property "Datasheet" ""
-			(at 302.26 142.24 0)
-			(effects
-				(font
-					(size 1.27 1.27)
-				)
-				(hide yes)
-			)
-		)
-		(property "Description" "Power symbol creates a global label with name \"+7.5V\""
-			(at 302.26 142.24 0)
-			(effects
-				(font
-					(size 1.27 1.27)
-				)
-				(hide yes)
-			)
-		)
-		(pin "1"
-		)
-		(instances
-			(project ""
-				(path "/af3cfa74-a4e1-440c-b447-a23ba1001a82/07efea5d-a0cf-4cd0-a91f-6ca432bf6d14"
-					(reference "#PWR0105")
-					(unit 1)
-				)
-			)
-		)
-	)
-	(symbol
 		(lib_id "power:GND")
 		(at 87.63 144.78 0)
@@
 			)
 		)
-		(property "Value" "1k"
+		(property "Value" "470"
 			(at 297.18 142.24 90)
 			(effects
@@
 			)
 		)
-		(property "Value" "470"
+		(property "Value" "680"
 			(at 203.454 36.068 90)
 			(effects

Commit message: メイン基板Rev.3
Parts:
- removed C22: 10uF, Capacitor_SMD:C_0603_1608Metric_Pad1.08x0.95mm_HandSolder, symbol Device:C
- removed C23: 22uF, Capacitor_SMD:C_0603_1608Metric_Pad1.08x0.95mm_HandSolder, symbol Device:C
- removed C24: 2.2uF, Capacitor_SMD:C_0805_2012Metric, symbol Device:C_Polarized
- removed C25: 470pF, Capacitor_SMD:C_0603_1608Metric_Pad1.08x0.95mm_HandSolder, symbol Device:C
- removed C26, C35, C37, C48: 4.7uF, Capacitor_SMD:C_0603_1608Metric_Pad1.08x0.95mm_HandSolder, symbol Device:C
- removed C27, C28, C29, C30, C31, C32, C33, C34, C38, C39, C40, C41, C42, C43, C44, C45, C46: 0.1uF, Capacitor_SMD:C_0603_1608Metric_Pad1.08x0.95mm_HandSolder, symbol Device:C
- removed C36, C47: 15pF, Capacitor_SMD:C_0603_1608Metric_Pad1.08x0.95mm_HandSolder, symbol Device:C
- removed D4: LED, LED_SMD:LED_0603_1608Metric, symbol Device:LED
- removed D5, D6, D7: WS2812B, LED_SMD:LED_WS2812B_PLCC4_5.0x5.0mm_P3.2mm, symbol LED:WS2812B
- removed J15: Comm to TopBoard, Connector_JST:JST_PH_B4B-PH-K_1x04_P2.00mm_Vertical, symbol Connector:Conn_01x04_Socket
- removed J16: Conn_01x08_Socket, Connector_PinSocket_2.54mm:PinSocket_1x08_P2.54mm_Vertical, symbol Connector:Conn_01x08_Socket
- removed J17, J18: ST-Link, STDC14:CONN14_3220-14_CNC, symbol Connector:Conn_ST_STDC14
- removed LS1: PKLCS1212E4001-R1, PKLCS1212E4001-R1:PKLCS1212E4001R1, symbol Device:Speaker
- removed M1, M2, M3, M4: STS3032, Connector_JST:JST_XH_B3B-XH-A_1x03_P2.50mm_Vertical, symbol STS3032:STS3032
- removed Q3: TJ15S06M3L, Package_TO_SOT_SMD:TO-252-2, symbol Simulation_SPICE:PMOS
- removed Q4, Q5: BSS138, Package_TO_SOT_SMD:SOT-23, symbol Simulation_SPICE:NMOS
- removed R17: 10k, Resistor_SMD:R_0603_1608Metric, symbol Device:R
- removed R18, R22: 680, Resistor_SMD:R_0603_1608Metric, symbol Device:R
- removed R19: 1k, Resistor_SMD:R_0603_1608Metric, symbol Device:R
- removed R20, R21, R23, R24, R25, R28: 10k, Capacitor_SMD:C_0603_1608Metric_Pad1.08x0.95mm_HandSolder, symbol Device:R
- removed R26: 470, Resistor_SMD:R_0603_1608Metric, symbol Device:R
- removed R27, R30, R31, R32, R33, R34: 2.2k, Capacitor_SMD:C_0603_1608Metric_Pad1.08x0.95mm_HandSolder, symbol Device:R
- removed SW3: B-12CCP, B-12CCP:B-12CCP, symbol B-12CCP:B-12CCP
- removed SW4, SW7: RESET_SWITCH, SKRPACE010:SW_SKRPACE010, symbol Switch:SW_Push
- removed SW5, SW8: MODE_SWITCH, SSSS213202:SSSS213202, symbol Switch:SW_DPDT_x2
- removed U10: AZ1117CH-3.3TRG1, AZ1117CH-3.3TRG1:DIODES_AZ1117CH-3.3TRG1_0, symbol AZ1117CH:AZ1117CH-3.3TRG1
- removed U11, U13: ~, Connector_PinSocket_2.54mm:PinSocket_1x06_P2.54mm_Vertical, symbol VL53l0X:VL53L0X_SwScience_6pin
- removed U12: AE-BNO055-BO, AE-BNO055-BO:AE-BNO055-BO, symbol AE-BNO055-BO:AE-BNO055-BO
- removed U14, U16: STM32F446RET6, Package_QFP:LQFP-64_10x10mm_P0.5mm, symbol MCU_ST_STM32F4:STM32F446RETx
- removed U15, U17: Sit2001B, Package_TO_SOT_SMD:SOT-23-5, symbol SiT2001B:Sit2001B
- removed U18: MAX3485, Package_SO:SOIC-8_3.9x4.9mm_P1.27mm, symbol Interface_UART:MAX3485
- removed U9: MIC5219-5.0YM5-TR, Package_TO_SOT_SMD:SOT-23-5, symbol MIC5219-5.0YM5-TR:MIC5219-5.0YM5-TR
- BT1: footprint Connector_AMASS:AMASS_XT30PW-F_1x02_P2.50mm_Horizontal -> Connector_AMASS:AMASS_XT30U-M_1x02_P5.0mm_Vertical
- J14: value Power to TopBoard -> Power to Main_Board; footprint Connector_AMASS:AMASS_XT30U-F_1x02_P5.0mm_Vertical -> Connector_AMASS:AMASS_XT30U-M_1x02_P5.0mm_Vertical
- R29: value 10k -> 3.3k; footprint Capacitor_SMD:C_0603_1608Metric_Pad1.08x0.95mm_HandSolder -> Resistor_SMD:R_0603_1608Metric
Connections:
- net +7.5V: now also R29.2
- net GND: no longer R29.1, SW6.3 (C)
- net at F1.2: now also SW6.2 (B)
- net VDD: now reaches SW6.1 (A)
- net at SW6.5 (A): now also R29.1
- no-connect marks 87 -> 1
Other:
- note added: "Power"
- note removed: "BL"
- note removed: "CK"
- note removed: "CS"
- note removed: "DC"
- note removed: "DISPLAY"
- note removed: "G"
- note removed: "MOTOR"
- note removed: "NEOPIXEL"
- note removed: "PH,Vertical"
- note removed: "POWER&COM"
- note removed: "PinHeader,Vertical"
- note removed: "RP-RX"
- note removed: "RP-TX"
- note removed: "RT"
- note removed: "SC"
- note removed: "SI"
- note removed: "SO"
- note removed: "SPEAKER"
- note removed: "ST-LINK"
- note removed: "STM-RX"
- note removed: "STM-TX"
- note removed: "STM32"
- note removed: "STM32 for UI"
- note removed: "TAJR225M016RNJ"
- note removed: "TOF"
- note removed: "V"
- note removed: "VBAT"
- note removed: "VDD"
- note removed: "VDDA"
- note removed: "XT30,Horizontal"
- company: Fornax -> (none)
- title: BackBoard Rev.2 -> (none)

Commit message: メイン基板Rev.3
Parts:
- added BT2: Battery, Connector_AMASS:AMASS_XT30PW-F_1x02_P2.50mm_Horizontal, symbol Device:Battery
- added F2: 0451015.MRL, 0451015.MRL:0451Series_LTF, symbol Device:Fuse
- added IC3: R3111N211A-TR-FE, R3111N211A:SOT95P280X130-5N, symbol R3111N211A:R3111N211A-TR-FE
- added MES2: Voltmeter_DC, Connector_JST:JST_XH_B2B-XH-A_1x02_P2.50mm_Vertical, symbol Device:Voltmeter_DC
- added Q1: TJ15S06M3L, Package_TO_SOT_SMD:TO-252-2, symbol Simulation_SPICE:PMOS
- added Q2: NMOS, symbol Simulation_SPICE:NMOS
- added R43, R47: 47k, Resistor_SMD:R_0603_1608Metric, symbol Device:R
- added R44: 5.6k, LED_SMD:LED_0402_1005Metric, symbol Device:R
- added R45: 470k, Resistor_SMD:R_0603_1608Metric, symbol Device:R
- added R46: 2.4k, LED_SMD:LED_0402_1005Metric, symbol Device:R
- added SW9: MODE_SWITCH, SSSS213202:SSSS213202, symbol Switch:SW_DPDT_x2
- renumbered J14 to J15, R29 to R28
Connections:
- net +7.5V: now also Q1.1 (D)
- net GND: now also BT2.2 (-), IC3.3 (GND), MES2.1 (-), Q2.3 (S), R45.1, R46.2
- new net: Q1.2 (G), Q2.1 (D), R43.1
- new net: F2.2, MES2.2 (+), Q1.3 (S), R43.2, R44.1, R47.2
- new net: BT2.1 (+), F2.1
- new net: IC3.2 (VDD), R44.2, R46.1
- new net: IC3.1 (OUT), Q2.2 (G), R45.2, SW9.2 (B)
- new net: R47.1, SW9.1 (A)
- no-connect marks 1 -> 2
Other:
- moved on the sheet: BT1, F1, MES1, R28, SW6

Commit message: 後ろ基板Rev.2
Parts:
- removed BT1: Battery, Connector_AMASS:AMASS_XT30U-M_1x02_P5.0mm_Vertical, symbol Device:Battery
- removed F1: 0451015.MRL, 0451015.MRL:0451Series_LTF, symbol Device:Fuse
- removed MES1: Voltmeter_DC, Connector_JST:JST_XH_B2B-XH-A_1x02_P2.50mm_Vertical, symbol Device:Voltmeter_DC
- removed Q2: NMOS, symbol Simulation_SPICE:NMOS
- removed R28: 3.3k, Resistor_SMD:R_0603_1608Metric, symbol Device:R
- removed SW6: B-12CCP, B-12CCP:B-12CCP, symbol B-12CCP:B-12CCP
- removed SW9: MODE_SWITCH, SSSS213202:SSSS213202, symbol Switch:SW_DPDT_x2
- added Q2, Q3: 2N7002, Package_TO_SOT_SMD:SOT-23, symbol Transistor_FET:2N7002
- added R44: R_Trim, 3362P-1-103LF:TRIM_3362P-1-103LF, symbol Device:R_Trim
- added SW5: START_SWITCH, B12AP_NKK:B12AP_NKK, symbol Switch:SW_SPDT
- BT1: renamed from BT2; footprint Connector_AMASS:AMASS_XT30PW-F_1x02_P2.50mm_Horizontal -> Connector_AMASS:AMASS_XT30U-M_1x02_P5.0mm_Vertical
- MES1: renamed from MES2; footprint Connector_JST:JST_XH_B2B-XH-A_1x02_P2.50mm_Vertical -> Connector_JST:JST_PH_B2B-PH-K_1x02_P2.00mm_Vertical
- R13: renamed from R44; value 5.6k -> 4.7k; footprint LED_SMD:LED_0402_1005Metric -> Resistor_SMD:R_0603_1608Metric_Pad0.98x0.95mm_HandSolder
- R28: renamed from R43; footprint Resistor_SMD:R_0603_1608Metric -> Resistor_SMD:R_0603_1608Metric_Pad0.98x0.95mm_HandSolder
- R43: renamed from R47; footprint Resistor_SMD:R_0603_1608Metric -> Resistor_SMD:R_0603_1608Metric_Pad0.98x0.95mm_HandSolder
- R45: value 470k -> 47k; footprint Resistor_SMD:R_0603_1608Metric -> Resistor_SMD:R_0603_1608Metric_Pad0.98x0.95mm_HandSolder
- R46: value 2.4k -> 470k; footprint LED_SMD:LED_0402_1005Metric -> Resistor_SMD:R_0603_1608Metric_Pad0.98x0.95mm_HandSolder
- renumbered F2 to F1
Connections:
- net GND: now also R46.1, Q3.2 (S), R44.2; no longer R45.1, R46.2
- net at Q1.2 (G), R28.1: now also Q2.3 (D)
- net at F1.2, MES1.2 (+), Q1.3 (S)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: now also R45.2
- net at IC3.2 (VDD), R13.2: now also R44.1; no longer R46.1
- net at IC3.1 (OUT): now also R43.1, Q2.1 (G); no longer R45.2
- new net: Q2.2 (S), Q3.3 (D)
- new net: R45.1, SW5.2 (B)
- new net: Q3.1 (G), R46.2, SW5.1 (A)
- no-connect marks 2 -> 1
Other:
- note added: "abt 2.2k"
- moved on the sheet: BT1, F1, IC3, MES1, Q1, R13, R28, R43
