File: TileBoard.kicad_sch (KiCad schematic)
At the start: 8 parts, among them J25 to TopBoard, U20 S11059

Commit message: Lidar基板Rev.2発注
Other:
- company: (none) -> Fornax
- title: (none) -> TileBoard Rev.1
Changed lines of the file:
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@@
 	(generator_version "8.0")
 	(paper "A5")
+	(title_block
+		(title "TileBoard Rev.1")
+		(rev "1")
+		(company "Fornax")
+	)
 	(junction
 		(at 172.72 30.48)

Commit message: メイン基板Rev.2完成
Parts:
- renumbered C74 to C64, D10 to D12, D11 to D13, J25 to J29, R41 to R43, R42 to R44, U20 to U23

Commit message: メイン基板Rev.3
Parts:
- removed A1: RPR-220, RPR-220:PHODET_RPR-220, symbol RPR-220:RPR-220
- removed C64: 0.1uF, Capacitor_SMD:C_0603_1608Metric, symbol Device:C
- removed D12: WS2812B, LED_SMD:LED_WS2812B_PLCC4_5.0x5.0mm_P3.2mm, symbol LED:WS2812B
- removed J29: to TopBoard, Connector_JST:JST_PH_B7B-PH-K_1x07_P2.00mm_Vertical, symbol Connector:Conn_01x07_Socket
- removed R43: 100, Capacitor_SMD:C_0603_1608Metric, symbol Device:R
- removed R44: 100k, Capacitor_SMD:C_0603_1608Metric, symbol Device:R
- removed U23: S11059, S11059:S11059, symbol S11059:S11059
- added C47: 0.1uF, Capacitor_SMD:C_0603_1608Metric, symbol Device:C
- added D14: WS2812B, LED_SMD:LED_WS2812B_PLCC4_5.0x5.0mm_P3.2mm, symbol LED:WS2812B
- added J19: to Main_Board, Connector_PinHeader_2.54mm:PinHeader_1x06_P2.54mm_Vertical, symbol Connector:Conn_01x06_Socket
- added R36, R37: 2.2k, Resistor_SMD:R_0603_1608Metric, symbol Device:R
- added U17: S11059, S11059:S11059, symbol S11059:S11059
Connections:
- net +3.3V: now also C47.1, J19.1 (Pin_1), R36.2, R37.2, U17.1 (VDD)
- net +5V: now also D14.1 (VDD), J19.2 (Pin_2)
- net GND: now also C47.2, D14.3 (VSS), J19.3 (Pin_3), U17.2 (GND)
- net IN: now also D13.4 (DIN), J19.6 (Pin_6)
- net SCL: now also J19.4 (Pin_4), R37.1, U17.3 (SCL)
- net SDA: now also J19.5 (Pin_5), R36.1, U17.4 (SDA)
- net at D13.2 (DOUT): now also D14.4 (DIN)
Other:
- note added: "Color_Sensor"
- note added: "LED"
- note added: "Power&Com"
- note removed: "COLOR_SENSOR"
- note removed: "NEOPIXEL"
- note removed: "PHOTO_REFLECTOR"
- note removed: "POWER&COM"
- company: Fornax -> (none)
- title: TileBoard Rev.1 -> (none)

Commit message: メイン基板Rev.3
Parts:
- renumbered C47 to C54, D13 to D14, D14 to D15, J19 to J20, R36 to R35, R37 to R36, U17 to U16
Changed lines of the file:
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@@
 	(label "IN"
 		(at 68.58 36.83 180)
+		(fields_autoplaced yes)
 		(effects
 			(font
@@
 	(label "SCL"
 		(at 40.64 38.1 0)
+		(fields_autoplaced yes)
 		(effects
 			(font
@@
 	(label "SCL"
 		(at 146.05 43.18 0)
+		(fields_autoplaced yes)
 		(effects
 			(font
@@
 	(label "SDA"
 		(at 139.7 39.37 0)
+		(fields_autoplaced yes)
 		(effects
 			(font
@@
 	(label "IN"
 		(at 40.64 43.18 0)
+		(fields_autoplaced yes)
 		(effects
 			(font
@@
 	(label "SDA"
 		(at 40.64 40.64 0)
+		(fields_autoplaced yes)
 		(effects
 			(font
@@
 		(on_board yes)
 		(dnp no)
-		(property "Reference" "#PWR0149"
+		(property "Reference" "#PWR0139"
 			(at 138.43 33.02 0)
 			(effects
@@
 			(project ""
 				(path "/b87cc2f7-3ac1-4af1-9a0e-9dfc79f9f7c4/4ccb1d87-a2eb-4440-a04b-5921d3896f33"
-					(reference "#PWR0149")
+					(reference "#PWR0139")
 					(unit 1)
 				)
@@
 		(dnp no)
 		(fields_autoplaced yes)
-		(property "Reference" "#PWR0147"
+		(property "Reference" "#PWR0137"
 			(at 77.47 29.21 0)
 			(effects
@@
 			(project "Final"
 				(path "/b87cc2f7-3ac1-4af1-9a0e-9dfc79f9f7c4/4ccb1d87-a2eb-4440-a04b-5921d3896f33"
-					(reference "#PWR0147")
+					(reference "#PWR0137")
 					(unit 1)
 				)
@@
 		(dnp no)
 		(fields_autoplaced yes)
-		(property "Reference" "#PWR0148"
+		(property "Reference" "#PWR0138"
 			(at 93.98 29.21 0)
 			(effects
@@
 			(project "Final"
 				(path "/b87cc2f7-3ac1-4af1-9a0e-9dfc79f9f7c4/4ccb1d87-a2eb-4440-a04b-5921d3896f33"
-					(reference "#PWR0148")
+					(reference "#PWR0138")
 					(unit 1)
 				)
@@
 		(on_board yes)
 		(dnp no)
-		(property "Reference" "#PWR0152"
+		(property "Reference" "#PWR0142"
 			(at 43.18 36.83 0)
 			(effects
@@
 			(project "Final"
 				(path "/b87cc2f7-3ac1-4af1-9a0e-9dfc79f9f7c4/4ccb1d87-a2eb-4440-a04b-5921d3896f33"
-					(reference "#PWR0152")
+					(reference "#PWR0142")
 					(unit 1)
 				)
@@
 		(on_board yes)
 		(dnp no)
-		(property "Reference" "#PWR0153"
+		(property "Reference" "#PWR0143"
 			(at 45.72 41.91 0)
 			(effects
@@
 			(project "Final"
 				(path "/b87cc2f7-3ac1-4af1-9a0e-9dfc79f9f7c4/4ccb1d87-a2eb-4440-a04b-5921d3896f33"
-					(reference "#PWR0153")
+					(reference "#PWR0143")
 					(unit 1)
 				)
@@
 		(dnp no)
 		(fields_autoplaced yes)
-		(property "Reference" "#PWR0156"
+		(property "Reference" "#PWR0146"
 			(at 77.47 53.34 0)
 			(effects
@@
 			(project "Final"
 				(path "/b87cc2f7-3ac1-4af1-9a0e-9dfc79f9f7c4/4ccb1d87-a2eb-4440-a04b-5921d3896f33"
-					(reference "#PWR0156")
+					(reference "#PWR0146")
 					(unit 1)
 				)
@@
 		(on_board yes)
 		(dnp no)
-		(property "Reference" "C47"
+		(property "Reference" "C54"
 			(at 112.268 39.624 0)
 			(effects
@@
 			(project "Final"
 				(path "/b87cc2f7-3ac1-4af1-9a0e-9dfc79f9f7c4/4ccb1d87-a2eb-4440-a04b-5921d3896f33"
-					(reference "C47")
+					(reference "C54")
 					(unit 1)
 				)
@@
 		(on_board yes)
 		(dnp no)
-		(property "Reference" "J19"
+		(property "Reference" "J20"
 			(at 33.655 25.4 0)
 			(effects
@@
 			(project ""
 				(path "/b87cc2f7-3ac1-4af1-9a0e-9dfc79f9f7c4/4ccb1d87-a2eb-4440-a04b-5921d3896f33"
-					(reference "J19")
+					(reference "J20")
 					(unit 1)
 				)
@@
 		(dnp no)
 		(fields_autoplaced yes)
-		(property "Reference" "#PWR0157"
+		(property "Reference" "#PWR0147"
 			(at 93.98 53.34 0)
 			(effects
@@
 			(project "Final"
 				(path "/b87cc2f7-3ac1-4af1-9a0e-9dfc79f9f7c4/4ccb1d87-a2eb-4440-a04b-5921d3896f33"
-					(reference "#PWR0157")
+					(reference "#PWR0147")
 					(unit 1)
 				)
@@
 		(on_board yes)
 		(dnp no)
-		(property "Reference" "#PWR0155"
+		(property "Reference" "#PWR0145"
 			(at 118.11 52.07 0)
 			(effects
@@
 			(project "Final"
 				(path "/b87cc2f7-3ac1-4af1-9a0e-9dfc79f9f7c4/4ccb1d87-a2eb-4440-a04b-5921d3896f33"
-					(reference "#PWR0155")
+					(reference "#PWR0145")
 					(unit 1)
 				)
@@
 		(on_board yes)
 		(dnp no)
-		(property "Reference" "#PWR0151"
+		(property "Reference" "#PWR0141"
 			(at 40.64 34.29 0)
 			(effects
@@
 			(project "Final"
 				(path "/b87cc2f7-3ac1-4af1-9a0e-9dfc79f9f7c4/4ccb1d87-a2eb-4440-a04b-5921d3896f33"
-					(reference "#PWR0151")
+					(reference "#PWR0141")
 					(unit 1)
 				)
@@
 		(on_board yes)
 		(dnp no)
-		(property "Reference" "#PWR0154"
+		(property "Reference" "#PWR0144"
 			(at 118.11 40.64 0)
 			(effects
@@
 			(project "Final"
 				(path "/b87cc2f7-3ac1-4af1-9a0e-9dfc79f9f7c4/4ccb1d87-a2eb-4440-a04b-5921d3896f33"
-					(reference "#PWR0154")
+					(reference "#PWR0144")
 					(unit 1)
 				)
@@
 		(on_board yes)
 		(dnp no)
-		(property "Reference" "#PWR0150"
+		(property "Reference" "#PWR0140"
 			(at 144.78 33.02 0)
 			(effects
@@
 			(project "Final"
 				(path "/b87cc2f7-3ac1-4af1-9a0e-9dfc79f9f7c4/4ccb1d87-a2eb-4440-a04b-5921d3896f33"
-					(reference "#PWR0150")
+					(reference "#PWR0140")
 					(unit 1)
 				)
@@
 		(on_board yes)
 		(dnp no)
-		(property "Reference" "D14"
+		(property "Reference" "D15"
 			(at 89.916 30.734 0)
 			(effects
@@
 			(project "Final"
 				(path "/b87cc2f7-3ac1-4af1-9a0e-9dfc79f9f7c4/4ccb1d87-a2eb-4440-a04b-5921d3896f33"
-					(reference "D14")
+					(reference "D15")
 					(unit 1)
 				)
@@
 		(on_board yes)
 		(dnp no)
-		(property "Reference" "U17"
+		(property "Reference" "U16"
 			(at 125.476 37.084 0)
 			(effects
@@
 			(project "Final"
 				(path "/b87cc2f7-3ac1-4af1-9a0e-9dfc79f9f7c4/4ccb1d87-a2eb-4440-a04b-5921d3896f33"
-					(reference "U17")
+					(reference "U16")
 					(unit 1)
 				)
@@
 		(on_board yes)
 		(dnp no)
-		(property "Reference" "D13"
+		(property "Reference" "D14"
 			(at 73.406 30.734 0)
 			(effects
@@
 			(project "Final"
 				(path "/b87cc2f7-3ac1-4af1-9a0e-9dfc79f9f7c4/4ccb1d87-a2eb-4440-a04b-5921d3896f33"
-					(reference "D13")
+					(reference "D14")
 					(unit 1)
 				)
@@
 		(on_board yes)
 		(dnp no)
-		(property "Reference" "R37"
+		(property "Reference" "R36"
 			(at 142.748 34.29 90)
 			(effects
@@
 			(project "Final"
 				(path "/b87cc2f7-3ac1-4af1-9a0e-9dfc79f9f7c4/4ccb1d87-a2eb-4440-a04b-5921d3896f33"
-					(reference "R37")
+					(reference "R36")
 					(unit 1)
 				)
@@
 		(on_board yes)
 		(dnp no)
-		(property "Reference" "R36"
+		(property "Reference" "R35"
 			(at 136.398 34.036 90)
 			(effects
@@
 			(project ""
 				(path "/b87cc2f7-3ac1-4af1-9a0e-9dfc79f9f7c4/4ccb1d87-a2eb-4440-a04b-5921d3896f33"
-					(reference "R36")
-					(unit 1)
-				)
+					(reference "R35")
+					(unit 1)
+				)
